File: calcvox.kicad_pcb (KiCad board)
At the start: 2 copper layers, 13 x 1.4 mm, 146 parts, among them J1 AudioJack2_Ground_Switch, SW1 RotaryEncoder_Switch, SW10 SW_Push, SW11 SW_Push, SW12 SW_Push, SW13 SW_Push, SW14 SW_Push, SW15 SW_Push, SW16 SW_Push, SW17 SW_Push, SW18 SW_Push, SW19 SW_Push, SW2 SW_Push, SW20 SW_Push, SW21 SW_Push, SW22 SW_Push, SW23 SW_Push, SW24 SW_Push, SW25 SW_Push, SW26 SW_Push, SW27 SW_Push, SW28 SW_Push, SW29 SW_Push, SW3 SW_Push, SW30 SW_Push, SW31 SW_Push, SW32 SW_Push, SW33 SW_Push, SW34 SW_Push, SW35 SW_Push, SW36 SW_Push, SW37 SW_Push, SW38 SW_Push, SW39 SW_Push, SW4 SW_Push, SW40 SW_Push, SW41 SW_Push, SW42 SW_Push, SW43 SW_Push, SW44 SW_Push, SW45 SW_Push, SW46 SW_Push, SW47 SW_Push, SW48 SW_Push, SW49 SW_Push, SW5 SW_Push, SW50 SW_Push, SW51 SW_Push, SW52 SW_Push, SW53 SW_Push, SW54 SW_Push, SW55 SW_Push, SW56 SW_Push, SW57 SW_Push, SW58 SW_Push, SW59 SW_Push, SW6 SW_Push, SW60 SW_Push, SW61 SW_Push, SW62 SW_Push, SW63 SW_Push, SW64 SW_Push, SW65 SW_Push, SW66 SW_Push, SW67 SW_SPDT, SW7 SW_Push, SW8 SW_Push, SW9 SW_Push

Commit message: added new changes
Parts:
- moved SW2 322.8 mm to (356.2, 292.2)
- moved D1 315.6 mm to (367.0, 279.4), turned to -90 degrees
- moved D2 279.9 mm to (367.0, 261.6), turned to -90 degrees
- moved D3 271.3 mm to (367.0, 242.6), turned to -90 degrees
- moved D4 263.7 mm to (367.0, 223.5), turned to -90 degrees
- moved D5 257.4 mm to (367.0, 203.2), turned to -90 degrees
- moved SW3 254.9 mm to (356.2, 274.3)
- moved D18 252.9 mm to (328.9, 261.6), turned to -90 degrees
- moved D6 252.6 mm to (367.0, 184.2), turned to -90 degrees
- moved D7 249.2 mm to (367.0, 165.1), turned to -90 degrees
- moved D8 247.3 mm to (367.0, 146.1), turned to -90 degrees
- moved SW4 246.0 mm to (356.2, 255.3)
- moved SW12 244.1 mm to (337.1, 255.3)
- moved D19 242.6 mm to (328.9, 242.6), turned to -90 degrees
- moved D9 239.7 mm to (348.0, 279.4), turned to -90 degrees
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